File: driver_40mm_atmega_v1p9/driver_40mm_atmega.kicad_pcb (KiCad board)
At the start: 6 copper layers, 40.4 x 40.4 mm, 424 parts, among them IC1 ATMEGA328P-M, IC2 ATMEGA328P-M, IC3 ATMEGA328P-M, IC4 ATMEGA328P-M, P1 CONN_2X2, P2 CONN_2X2, P3 CONN_2X2, P4 CONN_2X2, Q1 NMOS, Q10 NMOS, Q11 NMOS, Q12 NMOS, Q13 NMOS, Q14 NMOS, Q15 NMOS, Q16 NMOS, Q2 NMOS, Q3 NMOS, Q4 NMOS, Q5 NMOS, Q6 NMOS, Q7 NMOS, Q8 NMOS, Q9 NMOS, X1 20MHz, X2 20MHz, X3 20MHz, X4 20MHz

Commit message: add driver 1.9r5
Parts:
- D139: moved to B.Cu
- R10, R11, R12, R13, R14, R15, R16, R17, R18, R19, R20, R21, R22, R23, R24, R25, R26, R27, R28, R29, R30, R31, R32, R33, R34, R35, R36, R5, R6, R7, R8, R9: value 180 -> 240
- turned D139 to 135 degrees
Other:
- board text added: "2025-05-28"
- board text added: "G4.1 Driver v1.9.5"
- board text removed: "2024-07-29"
- board text removed: "G4.1 Driver v1.9.4"

Commit message: fix CPL file
Parts:
- D139: moved to F.Cu
- turned D139 to 45 degrees

Commit message: bump to 1.9.6, replace parts that are not available
Other:
- board text added: "${ISSUE_DATE}"
- board text added: "G4.1 Driver ${REVISION}"
- board text removed: "2025-05-28"
- board text removed: "G4.1 Driver v1.9.5"
Changed lines of the file:
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@@
 	(title_block
 		(title "G4.1 Driver 40mm ATMega")
-		(date "2025-05-28")
-		(rev "1.9.5")
+		(date "2025-07-31")
+		(rev "1.9.6")
 		(company "Reiser Lab @ Janelia")
 	)
@@
 		)
 		(embedded_fonts no)
-		(model "${KICAD6_3DMODEL_DIR}/Package_DFN_QFN.3dshapes/QFN-32-1EP_5x5mm_P0.5mm_EP3.1x3.1mm.wrl"
+		(model "${KIPRJMOD}/driver_custom.pretty/3dmodels/QFN-32-1EP_5x5mm_P0.5mm_EP3.7x3.7mm.step"
 			(offset
 				(xyz 0 0 0)
@@
 		)
 		(embedded_fonts no)
-		(model "${KICAD6_3DMODEL_DIR}/Package_DFN_QFN.3dshapes/QFN-32-1EP_5x5mm_P0.5mm_EP3.1x3.1mm.wrl"
+		(model "${KIPRJMOD}/driver_custom.pretty/3dmodels/QFN-32-1EP_5x5mm_P0.5mm_EP3.7x3.7mm.step"
 			(offset
 				(xyz 0 0 0)
@@
 		)
 		(embedded_fonts no)
-		(model "${KICAD6_3DMODEL_DIR}/Package_DFN_QFN.3dshapes/QFN-32-1EP_5x5mm_P0.5mm_EP3.1x3.1mm.wrl"
+		(model "${KIPRJMOD}/driver_custom.pretty/3dmodels/QFN-32-1EP_5x5mm_P0.5mm_EP3.7x3.7mm.step"
 			(offset
 				(xyz 0 0 0)
@@
 		)
 		(embedded_fonts no)
-		(model "${KICAD6_3DMODEL_DIR}/Package_DFN_QFN.3dshapes/QFN-32-1EP_5x5mm_P0.5mm_EP3.1x3.1mm.wrl"
+		(model "${KIPRJMOD}/driver_custom.pretty/3dmodels/QFN-32-1EP_5x5mm_P0.5mm_EP3.7x3.7mm.step"
 			(offset
 				(xyz 0 0 0)
@@
 		)
 	)
-	(gr_text "2025-05-28"
+	(gr_text "${ISSUE_DATE}"
 		(at 51.562 69.342 90)
 		(layer "B.SilkS")
@@
 		)
 	)
-	(gr_text "G4.1 Driver v1.9.5"
+	(gr_text "G4.1 Driver ${REVISION}"
 		(at 51.054 67.818 90)
 		(layer "B.SilkS")
