File: driver_40mm_atmega_v1p9/driver_40mm_atmega.kicad_pcb (KiCad board)
At the start: 6 copper layers, 40.4 x 40.4 mm, 424 parts, among them IC1 ATMEGA328P-M, IC2 ATMEGA328P-M, IC3 ATMEGA328P-M, IC4 ATMEGA328P-M, P1 CONN_2X2, P2 CONN_2X2, P3 CONN_2X2, P4 CONN_2X2, Q1 NMOS, Q10 NMOS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

Commit message: create driver v1.9.7
Parts:
- C10, C11, C12, C13, C14, C15, C16, C17, C18, C19, C20, C21, C22, C23, C24, C25, C26, C27, C28, C29, C30, C31, C32, C33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: value 200pF -> 220pF
