File: driver_40mm_atmega_v1p9/driver_40mm_atmega.kicad_sch (KiCad schematic)
At the start: 424 parts, among them IC1 ATMEGA328P-M, IC2 ATMEGA328P-M, IC3 ATMEGA328P-M, IC4 ATMEGA328P-M, P1 CONN_2X2, P2 CONN_2X2, P3 CONN_2X2, P4 CONN_2X2, Q1 NMOS, Q10 NMOS, Q11 NMOS, Q12 NMOS, Q13 NMOS, Q14 NMOS, Q15 NMOS, Q16 NMOS, Q2 NMOS, Q3 NMOS, Q4 NMOS, Q5 NMOS, Q6 NMOS, Q7 NMOS, Q8 NMOS, Q9 NMOS, X1 20MHz, X2 20MHz, X3 20MHz, X4 20MHz

Commit message: add driver 1.9r5
Parts:
- IC1, IC2, IC3, IC4, Q1, Q10, Q11, Q12, Q13, Q14, Q15, Q16, Q2, Q3, Q4, Q5, Q6, Q7, Q8, Q9: JLCPCB Rotation Offset (none) -> 90
- P1, P2, P3, P4: Alt JLCPCB 01 (none) -> C780055; Alt JLCPCB 02 (none) -> C7499901; JLCPCB PN C7499901 -> C919361; JLCPCB Rotation Offset (none) -> -90

Commit message: bump to 1.9.6, replace parts that are not available
Parts:
- C10, C11, C12, C13, C14, C15, C16, C17, C18, C19, C20, C21, C22, C23, C24, C25, C26, C27, C28, C29, C30, C31, C32, C33, C34, C35, C36, C5, C6, C7, C8, C9: value 200pF -> 220pF; JLCPCB PN C565508 -> C281748; PN FN03B221K160PLG -> CC0201KRX7R9BB221
- P1, P2, P3, P4: PN TSM-102-01-L-DV-P-TR -> 2.54-2*2P立贴针
- R10, R11, R12, R13, R14, R15, R16, R17, R18, R19, R20, R21, R22, R23, R24, R25, R26, R27, R28, R29, R30, R31, R32, R33, R34, R35, R36, R5, R6, R7, R8, R9: JLCPCB PN C166280 -> C155745; PN RTT012430FTH -> RC0201FR-07240RL
